File: motherboard.brd (EAGLE design)
At the start: 160 x 100 mm, 36 parts, among them IC1 93LCS56SN, IC2 93LCS56P, IC4 REG1117, IC5 NE555N, J1 J_ETHERNET_PULSE_J0011D01BNL

Commit message: production version
Parts:
- removed IC1: 93LCS56SN, microchip:SO-08
- removed IC2: 93LCS56P, microchip:DIL8
- added C10, C11, C7, C8, C9: (no value), rcl:C0805K
- added C6: 100n, rcl:C0805K
- added CAN: (no value), con-lstb:MA04-1
- added R13: 1k, rcl:R0805
- added SJ1, SJ2, SJ3, SJ5, SJ6, SJ7, SJ8: (no value), jumper:SJ
- added U1: TJA1050, NXP_60_26022015:SOT96-1
- added U2: 4MB Flash, SparkFun-IC-Memory:SO08
- C4: value (none) -> 100n
- R1, R2, R5, R6: value 49.9 -> 1k
- R7, R8: value 100 -> 1k
- moved UART0 149.9 mm to (6.35, 16.5), turned to 270 degrees
- moved R5 112.9 mm to (139.3, 84.7), turned to 180 degrees
- moved I2C0 72.8 mm to (118.1, 92.7), turned to 180 degrees
- moved R6 42.6 mm to (20.7, 12.8), turned to 0 degrees
- moved IC5 40.6 mm to (73.7, 11.4), turned to 0 degrees
- moved R2 29.7 mm to (33.0, 20.3), turned to 0 degrees
- moved R1 27.8 mm to (33.0, 17.8), turned to 180 degrees
- moved C4 19.1 mm to (25.4, 44.5), turned to 0 degrees
- moved 3V1 11.7 mm to (14.0, 33.0)
- moved 3V2 11.7 mm to (17.8, 33.0)
- moved 3V4 11.7 mm to (21.6, 33.0)
- moved R10 11.7 mm to (17.8, 27.9)
- moved R9 11.7 mm to (14.0, 27.9)
- moved 3V5 11.7 mm to (25.4, 33.0)
- moved R11 11.7 mm to (21.6, 27.9)
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Connections:
- removed net CS0: SPI0.6
- removed net N$390: U$1.P$41
- removed net N$391: U$1.P$40
- removed net N$392: U$1.P$39
- removed net N$393: U$1.P$38
- removed net N$63: U$1.P$9
- removed net SCK1\: SPI1.5
- removed net UART0_RX: UART0.3
- removed net UART0_TX: UART0.4
- removed net VCC: IC1.8, IC2.8
- new net CAN_H: CAN.3, U1.7
- new net CAN_L: CAN.4, U1.6
- new net CAN_RX: U$1.P$38, U1.4
- new net CAN_TX: U$1.P$39, U1.1
- new net CS_SPI_JUMPER: SPI0.3
- new net N$10: SJ2.2, SPI0.5
- new net N$11: SJ3.2, SPI0.4
- new net N$30: R13.2, R6.1, U1.8
- new net N$398: SJ6.2, SPI1.5
- new net N$399: SJ7.2, SPI1.4
- new net N$400: SJ8.2, SPI1.3
- new net N$9: SJ1.2, SPI0.6
- new net NOT_CS_FLASH: R5.1, U$1.P$9, U2.1
- new net UART_RX: U$1.P$41, UART0.3
- new net UART_TX: U$1.P$40, UART0.4
- net 3V3: now also C10.1, C11.1, C6.1, C9.1, R1.2, U2.8; no longer R1.1, R2.2, R5.2, R6.2
- net 5V0: now also C7.1, C8.1, CAN.2, R6.2, U1.3
- net CARD_CS: now also R2.2
- net CS1: now also SJ8.1, U$1.P$8; no longer SPI1.6
- net ETH_RX_N: no longer R6.1
- net ETH_RX_P: no longer R5.1
- net ETH_TX_N: no longer R2.1
- net ETH_TX_P: no longer R1.2
- net GND: now also C10.2, C11.2, C6.2, C7.2, C8.2, C9.2, CAN.1, R13.1, R2.1, R5.2, U1.2, U2.4; no longer IC1.5, IC2.5
- net LCD_CS: now also R1.1, U$1.P$21
- net MISO0: now also SJ3.1; no longer SPI0.3
- net MISO1: now also SJ7.1, U2.2; no longer SPI1.3
- net MOSI0: now also SJ1.1; no longer SPI0.4
- net MOSI1: now also SJ5.1, U2.5; no longer SPI1.4
- net N$376: now also SJ5.2, SPI1.6; no longer U$1.P$21
- net N$62: now also U2.7; no longer U$1.P$8
- net SCK0: now also SJ2.1; no longer SPI0.5
- net SCK1: now also SJ6.1, U2.6
Routing:
- net 5V0: track 34.1 -> 735.7 mm, vias 0 -> 48
- net 3V3: track 81.2 -> 772.6 mm, vias 4 -> 44
- net LCD_CS: track 0.00 -> 198.8 mm, vias 0 -> 1
- net MOSI0: track 0.00 -> 183.3 mm, vias 0 -> 3
- net MISO0: track 0.00 -> 179.2 mm, vias 0 -> 1
- net SCK0: track 0.00 -> 177.5 mm, vias 0 -> 3
- net CARD_CS: track 28.8 -> 194.9 mm, vias 3 -> 1
- net LCD_O/C: track 21.3 -> 186.7 mm, vias 2 -> 1
- net LCD_RST: track 36.4 -> 187.0 mm, vias 2 -> 1
- net UART_RX: track 0.00 -> 105.2 mm, vias 0 -> 1
- net N$4: track 2.54 -> 102.6 mm
- net UART_TX: track 0.00 -> 99.0 mm, vias 0 -> 1
- net I2C_SDA: track 2.54 -> 100.4 mm
- net SCK1: track 0.00 -> 97.4 mm, vias 0 -> 3
- net CAN_TX: track 0.00 -> 96.6 mm, vias 0 -> 1
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Other:
- board text added: "LPC 1769 Xpresso motherboard designed by Tomasz Lewicki, 2019"
