File: motherboard.sch (EAGLE design)
At the start: 36 parts, among them IC1 93LCS56SN, IC2 93LCS56P, IC4 REG1117, IC5 NE555N, J1 J_ETHERNET_PULSE_J0011D01BNL

Commit message: production version
Parts:
- removed IC1: 93LCS56SN, microchip:93LCS56SN
- removed IC2: 93LCS56P, microchip:93LCS56P
- added C10, C11, C7, C8, C9: (no value), rcl:C-EUC0805K
- added C6: 100n, rcl:C-EUC0805K
- added CAN: (no value), con-lstb:MA04-1
- added R13: 1k, rcl:R-EU_R0805
- added SJ1, SJ2, SJ3, SJ5, SJ6, SJ7, SJ8: (no value), jumper:SJ
- added U1: TJA1050, NXP_60_26022015:TJA1050
- added U2: 4MB Flash, SparkFun-IC-Memory:AT25SF041
- C4: value (none) -> 100n
- R1, R2, R5, R6: value 49.9 -> 1k
- R7, R8: value 100 -> 1k
Connections:
- removed net CS0: SPI0.6
- removed net N$390: U$1.P0.11
- removed net N$391: U$1.P0.10
- removed net N$392: U$1.P0.5
- removed net N$393: U$1.P0.4
- removed net N$63: U$1.P0.0
- removed net SCK1\: SPI1.5
- removed net UART0_RX: UART0.3
- removed net UART0_TX: UART0.4
- new net CAN_H: CAN.3, U1.CANH
- new net CAN_L: CAN.4, U1.CANL
- new net CAN_RX: U$1.P0.4, U1.RXD
- new net CAN_TX: U$1.P0.5, U1.TXD
- new net CS_SPI_JUMPER: SPI0.3
- new net N$10: SJ2.2, SPI0.5
- new net N$11: SJ3.2, SPI0.4
- new net N$30: R13.2, R6.1, U1.S
- new net N$398: SJ6.2, SPI1.5
- new net N$399: SJ7.2, SPI1.4
- new net N$400: SJ8.2, SPI1.3
- new net N$9: SJ1.2, SPI0.6
- new net NOT_CS_FLASH: R5.1, U$1.P0.0, U2.!CS
- new net UART_RX: U$1.P0.11, UART0.3
- new net UART_TX: U$1.P0.10, UART0.4
- net 3V3: now also C10.1, C11.1, C6.1, C9.1, R1.2, U2.VCC; no longer R1.1, R2.2, R5.2, R6.2
- net 5V0: now also C7.1, C8.1, CAN.2, R6.2, U1.VCC
- net CARD_CS: now also R2.2
- net CS1: now also SJ8.1, U$1.P0.6; no longer SPI1.6
- net ETH_RX_N: no longer R6.1
- net ETH_RX_P: no longer R5.1
- net ETH_TX_N: no longer R2.1
- net ETH_TX_P: no longer R1.2
- net GND: now also C10.2, C11.2, C6.2, C7.2, C8.2, C9.2, CAN.1, R13.1, R2.1, R5.2, U1.GND, U2.GND
- net LCD_CS: now also R1.1, U$1.P0.2
- net MISO0: now also SJ3.1; no longer SPI0.3
- net MISO1: now also SJ7.1, U2.SO; no longer SPI1.3
- net MOSI0: now also SJ1.1; no longer SPI0.4
- net MOSI1: now also SJ5.1, U2.SI; no longer SPI1.4
- net N$376: now also SJ5.2, SPI1.6; no longer U$1.P0.2
- net N$62: now also U2.!HOLD; no longer U$1.P0.6
- net SCK0: now also SJ2.1; no longer SPI0.5
- net SCK1: now also SJ6.1, U2.SCK
Other:
- note added: "external power"
- moved on the sheet: C4, C5, CN2, IC4, R7, R8
